File: hardware/joystick-v2.kicad_pcb (KiCad board)
At the start: 2 copper layers, 45 x 25 mm, 23 parts, among them P1 CON-SENSOR2, P2 DEBUG, P3 BOOT, U1 XMC1XXX24, U3 JOYSTICK_BUTTON, U4 DRILL, U5 DRILL, U6 DRILL, U7 DRILL

Commit message: fixed lib, added sym_lib_table, changed processor to XMC1100
Parts:
- U1: value XMC1XXX24 -> XMC1100
Changed lines of the file:
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@@
       (effects (font (size 0.3 0.3) (thickness 0.075)))
     )
-    (fp_text value XMC1XXX24 (at 0 0.8 270) (layer F.Fab)
+    (fp_text value XMC1100 (at 0 0.8 270) (layer F.Fab)
       (effects (font (size 0.3 0.3) (thickness 0.075)))
     )
